File: PCB/nixie-3-board/nixie-3-board.kicad_sch (KiCad schematic)
At the start: 21 parts, among them J1 Conn_01x07_Socket, J2 Conn_01x07_Pin, J3 SFH11-PBPC-D07-ST-BK, J4 SFH11-PBPC-D07-ST-BK, Q1 MPSA92, Q4 MPSA42, U1 74HC595, U2 74141, U3 74141

Commit message: Fixed mistakes, v3.1
Parts:
- added H4: MountingHole, MountingHole:MountingHole_2.7mm_M2.5_DIN965, symbol Mechanical:MountingHole
Other:
- moved on the sheet: H1, H2, H3
Changed lines of the file:
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@@
     )
   )
-  (symbol (lib_id "Mechanical:MountingHole") (at 26.035 41.91 0) (unit 1)
-    (in_bom yes) (on_board yes) (dnp no) (fields_autoplaced)
-    (property "Reference" "H2" (at 29.21 40.64 0)
-      (effects (font (size 1.27 1.27)) (justify left))
-    )
-    (property "Value" "MountingHole" (at 29.21 43.18 0)
-      (effects (font (size 1.27 1.27)) (justify left))
-    )
-    (property "Footprint" "MountingHole:MountingHole_2.7mm_M2.5_DIN965" (at 26.035 41.91 0)
-      (effects (font (size 1.27 1.27)) hide)
-    )
-    (property "Datasheet" "~" (at 26.035 41.91 0)
+  (symbol (lib_id "Mechanical:MountingHole") (at 25.4 32.385 0) (unit 1)
+    (in_bom yes) (on_board yes) (dnp no) (fields_autoplaced)
+    (property "Reference" "H2" (at 28.575 31.115 0)
+      (effects (font (size 1.27 1.27)) (justify left))
+    )
+    (property "Value" "MountingHole" (at 28.575 33.655 0)
+      (effects (font (size 1.27 1.27)) (justify left))
+    )
+    (property "Footprint" "MountingHole:MountingHole_2.7mm_M2.5_DIN965" (at 25.4 32.385 0)
+      (effects (font (size 1.27 1.27)) hide)
+    )
+    (property "Datasheet" "~" (at 25.4 32.385 0)
       (effects (font (size 1.27 1.27)) hide)
     )
@@
     )
   )
-  (symbol (lib_id "Mechanical:MountingHole") (at 26.035 35.56 0) (unit 1)
-    (in_bom yes) (on_board yes) (dnp no) (fields_autoplaced)
-    (property "Reference" "H1" (at 29.21 34.29 0)
-      (effects (font (size 1.27 1.27)) (justify left))
-    )
-    (property "Value" "MountingHole" (at 29.21 36.83 0)
-      (effects (font (size 1.27 1.27)) (justify left))
-    )
-    (property "Footprint" "MountingHole:MountingHole_2.7mm_M2.5_DIN965" (at 26.035 35.56 0)
-      (effects (font (size 1.27 1.27)) hide)
-    )
-    (property "Datasheet" "~" (at 26.035 35.56 0)
+  (symbol (lib_id "Mechanical:MountingHole") (at 25.4 26.035 0) (unit 1)
+    (in_bom yes) (on_board yes) (dnp no) (fields_autoplaced)
+    (property "Reference" "H1" (at 28.575 24.765 0)
+      (effects (font (size 1.27 1.27)) (justify left))
+    )
+    (property "Value" "MountingHole" (at 28.575 27.305 0)
+      (effects (font (size 1.27 1.27)) (justify left))
+    )
+    (property "Footprint" "MountingHole:MountingHole_2.7mm_M2.5_DIN965" (at 25.4 26.035 0)
+      (effects (font (size 1.27 1.27)) hide)
+    )
+    (property "Datasheet" "~" (at 25.4 26.035 0)
       (effects (font (size 1.27 1.27)) hide)
     )
@@
     )
   )
-  (symbol (lib_id "Mechanical:MountingHole") (at 26.035 48.26 0) (unit 1)
-    (in_bom yes) (on_board yes) (dnp no) (fields_autoplaced)
-    (property "Reference" "H3" (at 29.21 46.99 0)
-      (effects (font (size 1.27 1.27)) (justify left))
-    )
-    (property "Value" "MountingHole" (at 29.21 49.53 0)
-      (effects (font (size 1.27 1.27)) (justify left))
-    )
-    (property "Footprint" "MountingHole:MountingHole_2.7mm_M2.5_DIN965" (at 26.035 48.26 0)
-      (effects (font (size 1.27 1.27)) hide)
-    )
-    (property "Datasheet" "~" (at 26.035 48.26 0)
+  (symbol (lib_id "Mechanical:MountingHole") (at 25.4 38.735 0) (unit 1)
+    (in_bom yes) (on_board yes) (dnp no) (fields_autoplaced)
+    (property "Reference" "H3" (at 28.575 37.465 0)
+      (effects (font (size 1.27 1.27)) (justify left))
+    )
+    (property "Value" "MountingHole" (at 28.575 40.005 0)
+      (effects (font (size 1.27 1.27)) (justify left))
+    )
+    (property "Footprint" "MountingHole:MountingHole_2.7mm_M2.5_DIN965" (at 25.4 38.735 0)
+      (effects (font (size 1.27 1.27)) hide)
+    )
+    (property "Datasheet" "~" (at 25.4 38.735 0)
       (effects (font (size 1.27 1.27)) hide)
     )
@@
         )
       )
+    )
+  )
+  (symbol (lib_id "Mechanical:MountingHole") (at 25.4 45.085 0) (unit 1)
+    (in_bom yes) (on_board yes) (dnp no) (fields_autoplaced)
+    (property "Reference" "H4" (at 28.575 43.815 0)
+      (effects (font (size 1.27 1.27)) (justify left))
+    )
+    (property "Value" "MountingHole" (at 28.575 46.355 0)
+      (effects (font (size 1.27 1.27)) (justify left))
+    )
+    (property "Footprint" "MountingHole:MountingHole_2.7mm_M2.5_DIN965" (at 25.4 45.085 0)
+      (effects (font (size 1.27 1.27)) hide)
+    )
+    (property "Datasheet" "~" (at 25.4 45.085 0)
+      (effects (font (size 1.27 1.27)) hide)
+    )
+    (instances
+      (project "nixie-3-board"
+        (path "/fbd11439-5a75-46fa-bc19-b9f5c38db8a0"
+          (reference "H4") (unit 1)
+        )
+      )

Commit message: Better names for the decoupling cap footprint files
Also corrected the value for the PS decoupling cap from 100uF to 10uF
Parts:
- C4: value 100µF -> 10µF
Changed lines of the file:
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@@
       (effects (font (size 1.27 1.27)) (justify left))
     )
-    (property "Value" "100µF" (at 86.36 161.925 0)
+    (property "Value" "10µF" (at 86.36 161.925 0)
       (effects (font (size 1.27 1.27)) (justify left))
     )

Commit message: Removed unused INPUT_SWITCH, dropped PORTB use by the RTC
Other:
- note added: "Note: R4 at 7.5k with HV at 175v has 32v across it --> The two tubes are getting 4.27mA. For DC operation, they should get 1mA, so this resistor should be increased to 15k - 20k. 15k --> 1.07mA/Tube, 20k --> 0.8mA/Tube."
