File: PCB/nixie-3-board/nixie-3-board.kicad_sch (KiCad schematic)
At the start: 22 parts, among them J1 Conn_01x07_Socket, J2 Conn_01x07_Pin, J3 SFH11-PBPC-D07-ST-BK, J4 SFH11-PBPC-D07-ST-BK, Q1 MPSA92, Q4 MPSA42, U1 74HC595, U2 74141, U3 74141

Commit message: Moved docs to hv-ps-docs for the claude swe framework
Parts:
- renumbered Q4 to Q1, Q1 to Q2, R10 to R1, R1 to R2, R4 to R3, R7 to R4, R13 to R5
