File: PCB/555-HV-PS/555-HV-PS/555-HV-PS.kicad_sch (KiCad schematic)
At the start: 32 parts, among them J1 Barrel_Jack_Switch, J2 Conn_3_screw, Q1 2N2222, Q2 IRF730-TO-220-3, U1 LM7805_TO220, U2 LM555xN

Commit message: Edits to the 555 HV PS circuit and added some info
I added a README to the PCB/555-HV-PS directory with some
images from  the ocilloscope.
Parts:
- removed C4: 100pF, Capacitor_THT:C_Disc_D4.3mm_W1.9mm_P5.00mm, symbol HV-PS:C
- removed R2: 1M, Resistor_THT:R_Axial_DIN0207_L6.3mm_D2.5mm_P10.16mm_Horizontal, symbol HV-PS:R
- added R5: 3.3K, Resistor_THT:R_Axial_DIN0207_L6.3mm_D2.5mm_P10.16mm_Horizontal, symbol HV-PS:R
- C9: value 0.1uF -> 470pF
- L1: value 100uH 900mA -> 100uH 900mOhm
- R1: value 56k -> 33k
- renumbered C6 to C1, C8 to C2, C1 to C4, C2 to C5, C7 to C6, C5 to C7, C3 to C8, R6 to R2, R7 to R3, R3 to R4, R4 to R6, R5 to R7, U2 to U1, U1 to U2
Connections:
- net HV V out: no longer C9.1
- net at CR1.2, L1.1, Q2.2 (D): now also R5.1
- new net: C9.1, R5.2
Other:
- note added: "1. C6 Improves efficency by reducing current from the +12/15V supply by 10mA. 2. The sunubber network (R5, C9) reduces ringing in HV Vout."
- note added: "Notes"
- note removed: "FIXME C9"
- title: HV-PS-2, 15 to 180v, Using a 555  -> HV-PS-2, 12 to 177v, Using a 555 
- moved on the sheet: C6, CR1
