File: PCB/555-HV-PS/555-HV-PS/555-HV-PS.kicad_sch (KiCad schematic)
At the start: 31 parts, among them J1 Barrel_Jack_Switch, J2 Conn_3_screw, Q1 2N2222, Q2 IRF730-TO-220-3, U1 LM555xN, U2 LM7805_TO220

Commit message: Moved docs to hv-ps-docs for the claude swe framework
Changed lines of the file:
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@@
 (kicad_sch
-	(version 20231120)
+	(version 20250114)
 	(generator "eeschema")
-	(generator_version "8.0")
+	(generator_version "9.0")
 	(paper "USLetter")
 	(title_block
@@
 		(comment 3 "V1: 2024-12-23")
 	)
+	(rectangle
+		(start 128.27 90.17)
+		(end 259.08 166.37)
+		(stroke
+			(width 0)
+			(type default)
+		)
+		(fill
+			(type none)
+		)
+	)
+	(rectangle
+		(start 30.48 182.245)
+		(end 116.205 199.39)
+		(stroke
+			(width 0)
+			(type default)
+		)
+		(fill
+			(type none)
+		)
+	)
+	(rectangle
+		(start 33.02 83.82)
+		(end 106.68 128.27)
+		(stroke
+			(width 0)
+			(type default)
+		)
+		(fill
+			(type none)
+		)
+	)
+	(rectangle
+		(start 128.27 17.145)
+		(end 241.935 86.36)
+		(stroke
+			(width 0)
+			(type default)
+		)
+		(fill
+			(type none)
+		)
+	)
+	(text "1. C6 Improves efficency by reducing current from the +12/15V supply by 10mA.\n2. The sunubber network (R5, C9) reduces ringing in HV Vout."
+		(exclude_from_sim no)
+		(at 33.274 187.706 0)
+		(effects
+			(font
+				(size 1.27 1.27)
+			)
+			(justify left)
+		)
+	)
+	(text "Notes"
+		(exclude_from_sim no)
+		(at 68.072 195.834 0)
+		(effects
+			(font
+				(size 1.905 1.905)
+			)
+		)
+	)
+	(text "15V Power In"
+		(exclude_from_sim no)
+		(at 50.8 71.12 0)
+		(effects
+			(font
+				(size 3.81 3.81)
+			)
+			(justify left bottom)
+		)
+	)
+	(text "HV"
+		(exclude_from_sim no)
+		(at 187.96 162.56 0)
+		(effects
+			(font
+				(size 3.81 3.81)
+			)
+		)
+	)
+	(text "HV Control"
+		(exclude_from_sim no)
+		(at 185.42 81.28 0)
+		(effects
+			(font
+				(size 3.81 3.81)
+			)
+		)
+	)
+	(text "5V Power Out"
+		(exclude_from_sim no)
+		(at 50.292 125.476 0)
+		(effects
+			(font
+				(size 3.81 3.81)
+			)
+			(justify left bottom)
+		)
+	)
 	(junction
 		(at 55.88 50.8)
@@
 		)
 	)
-	(rectangle
-		(start 128.27 90.17)
-		(end 259.08 166.37)
-		(stroke
-			(width 0)
-			(type default)
-		)
-		(fill
-			(type none)
-		)
-	)
-	(rectangle
-		(start 30.48 182.245)
-		(end 116.205 199.39)
-		(stroke
-			(width 0)
-			(type default)
-		)
-		(fill
-			(type none)
-		)
-	)
-	(rectangle
-		(start 33.02 83.82)
-		(end 106.68 128.27)
-		(stroke
-			(width 0)
-			(type default)
-		)
-		(fill
-			(type none)
-		)
-	)
-	(rectangle
-		(start 128.27 17.145)
-		(end 241.935 86.36)
-		(stroke
-			(width 0)
-			(type default)
-		)
-		(fill
-			(type none)
-		)
-	)
-	(text "1. C6 Improves efficency by reducing current from the +12/15V supply by 10mA.\n2. The sunubber network (R5, C9) reduces ringing in HV Vout."
-		(exclude_from_sim no)
-		(at 33.274 187.706 0)
-		(effects
-			(font
-				(size 1.27 1.27)
-			)
-			(justify left)
-		)
-	)
-	(text "Notes"
-		(exclude_from_sim no)
-		(at 68.072 195.834 0)
-		(effects
-			(font
-				(size 1.905 1.905)
-			)
-		)
-	)
-	(text "15V Power In"
-		(exclude_from_sim no)
-		(at 50.8 71.12 0)
-		(effects
-			(font
-				(size 3.81 3.81)
-			)
-			(justify left bottom)
-		)
-	)
-	(text "HV"
-		(exclude_from_sim no)
-		(at 187.96 162.56 0)
-		(effects
-			(font
-				(size 3.81 3.81)
-			)
-		)
-	)
-	(text "HV Control"
-		(exclude_from_sim no)
-		(at 185.42 81.28 0)
-		(effects
-			(font
-				(size 3.81 3.81)
-			)
-		)
-	)
-	(text "5V Power Out"
-		(exclude_from_sim no)
-		(at 50.292 125.476 0)
-		(effects
-			(font
-				(size 3.81 3.81)
-			)
-			(justify left bottom)
-		)
-	)
 	(global_label "HV V out"
 		(shape output)
@@
 		)
 	)
+	(embedded_fonts no)
 )
